File: APRL_BMS_DEV_PCB.kicad_pcb (KiCad board)
At the start: 2 copper layers, 2 parts, among them U1 BQ756506-Q1, U2 STM32F446RCTx

Commit message: More
Connections:
- U1 pad 36: unconnected-(U1-REFHM-Pad36) -> GND
- U1 pad 39: unconnected-(U1-AVSS-Pad39) -> GND
- U1 pad 46: unconnected-(U1-CVSS-Pad46) -> GND
- U1 pad 50: unconnected-(U1-DVSS-Pad50) -> GND
- U2 pad 1: unconnected-(U2-VBAT-Pad1) -> +3.3V
- U2 pad 12: unconnected-(U2-VSSA-Pad12) -> GND
- U2 pad 13: unconnected-(U2-VDDA-Pad13) -> +3.3VA
- U2 pad 14: unconnected-(U2-PA0-Pad14) -> /UART_TX
- U2 pad 15: unconnected-(U2-PA1-Pad15) -> /UART_RX
- U2 pad 18: Net-(U2-VSS-Pad18) -> GND
- U2 pad 19: unconnected-(U2-VDD-Pad19) -> +3.3V
- U2 pad 31: Net-(U2-VSS-Pad18) -> GND
- U2 pad 32: unconnected-(U2-VDD-Pad32) -> +3.3V
- U2 pad 33: unconnected-(U2-PB12-Pad33) -> /CAN2_RX
- U2 pad 34: unconnected-(U2-PB13-Pad34) -> /CAN2_TX
- U2 pad 44: unconnected-(U2-PA11-Pad44) -> /CAN1_RX
- U2 pad 45: unconnected-(U2-PA12-Pad45) -> /CAN1_TX
- U2 pad 46: unconnected-(U2-PA13-Pad46) -> /SWDIO
- U2 pad 47: Net-(U2-VSS-Pad18) -> GND
- U2 pad 48: unconnected-(U2-VDD-Pad48) -> +3.3V
- U2 pad 49: unconnected-(U2-PA14-Pad49) -> /SWCLK
- U2 pad 5: unconnected-(U2-PH0-Pad5) -> Net-(U2-PH0)
- U2 pad 6: unconnected-(U2-PH1-Pad6) -> Net-(U2-PH1)
- U2 pad 60: unconnected-(U2-BOOT0-Pad60) -> /BOOT0
- U2 pad 63: Net-(U2-VSS-Pad18) -> GND
- U2 pad 64: unconnected-(U2-VDD-Pad64) -> +3.3V
- U2 pad 7: unconnected-(U2-NRST-Pad7) -> /NRST

Commit message: Added initial footprints and values for caps
Other:
- copper layers 2 -> 4
Changed lines of the file:
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@@
 	(layers
 		(0 "F.Cu" signal)
+		(4 "In1.Cu" signal)
+		(6 "In2.Cu" signal)
 		(2 "B.Cu" signal)
 		(9 "F.Adhes" user "F.Adhesive")
@@
 	)
 	(setup
+		(stackup
+			(layer "F.SilkS"
+				(type "Top Silk Screen")
+			)
+			(layer "F.Paste"
+				(type "Top Solder Paste")
+			)
+			(layer "F.Mask"
+				(type "Top Solder Mask")
+				(thickness 0.01)
+			)
+			(layer "F.Cu"
+				(type "copper")
+				(thickness 0.035)
+			)
+			(layer "dielectric 1"
+				(type "prepreg")
+				(thickness 0.1)
+				(material "FR4")
+				(epsilon_r 4.5)
+				(loss_tangent 0.02)
+			)
+			(layer "In1.Cu"
+				(type "copper")
+				(thickness 0.035)
+			)
+			(layer "dielectric 2"
+				(type "core")
+				(thickness 1.24)
+				(material "FR4")
+				(epsilon_r 4.5)
+				(loss_tangent 0.02)
+			)
+			(layer "In2.Cu"
+				(type "copper")
+				(thickness 0.035)
+			)
+			(layer "dielectric 3"
+				(type "prepreg")
+				(thickness 0.1)
+				(material "FR4")
+				(epsilon_r 4.5)
+				(loss_tangent 0.02)
+			)
+			(layer "B.Cu"
+				(type "copper")
+				(thickness 0.035)
+			)
+			(layer "B.Mask"
+				(type "Bottom Solder Mask")
+				(thickness 0.01)
+			)
+			(layer "B.Paste"
+				(type "Bottom Solder Paste")
+			)
+			(layer "B.SilkS"
+				(type "Bottom Silk Screen")
+			)
+			(copper_finish "None")
+			(dielectric_constraints no)
+		)
 		(pad_to_mask_clearance 0)
 		(allow_soldermask_bridges_in_footprints no)
